Commit message: Update launch files and URDF for multi-robot support

File: src/path_planning/urdf/robot_1.urdf (robot description, URDF)
Before this commit: robot robot_1, 2 links, 1 joints
Links:
- added link back_left_wheel_link, mass 0.5; collision cylinder length=0.05 radius=0.05; visual cylinder length=0.05 radius=0.05
- added link back_right_wheel_link, mass 0.5; collision cylinder length=0.05 radius=0.05; visual cylinder length=0.05 radius=0.05
- added link front_left_wheel_link, mass 0.5; collision cylinder length=0.05 radius=0.05; visual cylinder length=0.05 radius=0.05
- added link front_right_wheel_link, mass 0.5; collision cylinder length=0.05 radius=0.05; visual cylinder length=0.05 radius=0.05
Joints:
- added joint back_left_wheel_joint: type continuous, parent base_link, child back_left_wheel_link, origin xyz=-0.15 0.15 -0.1 rpy=0 0 0, axis 0 1 0
- added joint back_right_wheel_joint: type continuous, parent base_link, child back_right_wheel_link, origin xyz=-0.15 -0.15 -0.1 rpy=0 0 0, axis 0 1 0
- added joint front_left_wheel_joint: type continuous, parent base_link, child front_left_wheel_link, origin xyz=0.15 0.15 -0.1 rpy=0 0 0, axis 0 1 0
- added joint front_right_wheel_joint: type continuous, parent base_link, child front_right_wheel_link, origin xyz=0.15 -0.15 -0.1 rpy=0 0 0, axis 0 1 0

Commit message: 자율주행 코드 수정

File: src/path_planning/urdf/robot_1.urdf (robot description, URDF)
Before this commit: robot robot_1, 6 links, 5 joints
Links:
- added link base_footprint
Joints:
- added joint base_footprint_to_base_link: type fixed, parent base_footprint, child base_link, origin xyz=0 0 0 rpy=0 0 0
- joint back_left_wheel_joint: type continuous -> fixed

Commit message: 프젝에 끝이 있을까요?

File: src/path_planning/urdf/robot_1.urdf (robot description, URDF)
Before this commit: robot robot_1, 7 links, 6 joints
Joints:
- joint back_right_wheel_joint: type continuous -> fixed
- joint lidar_joint: origin xyz=0 0 0.15 rpy=0 0 0 -> xyz=0.2 0 0.12 rpy=0 0 0
